File: hardware/HifiPlayer.sch (KiCad schematic (older format))
At the start: 9 parts

Commit message: First layout
Parts:
- C1, C3: renamed from C?; footprint (none) -> Capacitor_SMD:C_1206_3216Metric_Pad1.42x1.75mm_HandSolder
- C2: renamed from C?; footprint (none) -> Capacitor_THT:CP_Radial_D5.0mm_P2.00mm
- J1: renamed from J?; footprint (none) -> Connector_PinHeader_2.54mm:PinHeader_1x04_P2.54mm_Vertical
- J2: renamed from J?; footprint (none) -> Connector_PinHeader_2.54mm:PinHeader_1x03_P2.54mm_Vertical
- J3: renamed from J?; footprint (none) -> Connector_PinHeader_2.54mm:PinHeader_1x06_P2.54mm_Vertical
- J4: renamed from J?; footprint (none) -> TerminalBlock:TerminalBlock_bornier-3_P5.08mm
- J5: renamed from J?; footprint (none) -> Connector_PinHeader_2.54mm:PinHeader_1x02_P2.54mm_Vertical
- gave numbers to parts that had none: 1
Changed lines of the file:
@@
 $EndDescr
 $Comp
-L MCU_ST_STM32G0:STM32G071KBTx U?
+L MCU_ST_STM32G0:STM32G071KBTx U1
 U 1 1 5E7CDB46
 P 4400 4350
-F 0 "U?" H 3950 5250 50  0000 C CNN
+F 0 "U1" H 3950 5250 50  0000 C CNN
 F 1 "STM32G071KBTx" H 4800 5250 50  0000 C CNN
 F 2 "Package_QFP:LQFP-32_7x7mm_P0.8mm" H 3200 2800 50  0001 C CNN
@@
 $EndComp
 $Comp
-L power:+3.3V #PWR?
+L power:+3.3V #PWR0101
 U 1 1 5E7D0C55
 P 4400 3300
-F 0 "#PWR?" H 4400 3150 50  0001 C CNN
+F 0 "#PWR0101" H 4400 3150 50  0001 C CNN
 F 1 "+3.3V" H 4415 3473 50  0000 C CNN
 F 2 "" H 4400 3300 50  0001 C CNN
@@
 	4400 3300 4400 3400
 $Comp
-L power:GND #PWR?
+L power:GND #PWR0102
 U 1 1 5E7D1E28
 P 4400 5500
-F 0 "#PWR?" H 4400 5250 50  0001 C CNN
+F 0 "#PWR0102" H 4400 5250 50  0001 C CNN
 F 1 "GND" H 4405 5327 50  0000 C CNN
 F 2 "" H 4400 5500 50  0001 C CNN
@@
 	4400 5400 4400 5500
 $Comp
-L power:+3.3V #PWR?
+L power:+3.3V #PWR0103
 U 1 1 5E7D290C
 P 1700 1300
-F 0 "#PWR?" H 1700 1150 50  0001 C CNN
+F 0 "#PWR0103" H 1700 1150 50  0001 C CNN
 F 1 "+3.3V" H 1715 1473 50  0000 C CNN
 F 2 "" H 1700 1300 50  0001 C CNN
@@
 $EndComp
 $Comp
-L power:GND #PWR?
+L power:GND #PWR0104
 U 1 1 5E7D35E6
 P 1700 1800
-F 0 "#PWR?" H 1700 1550 50  0001 C CNN
+F 0 "#PWR0104" H 1700 1550 50  0001 C CNN
 F 1 "GND" H 1705 1627 50  0000 C CNN
 F 2 "" H 1700 1800 50  0001 C CNN
@@
 $EndComp
 $Comp
-L Device:C C?
+L Device:C C1
 U 1 1 5E7D3EA0
 P 1700 1550
-F 0 "C?" H 1815 1596 50  0000 L CNN
+F 0 "C1" H 1815 1596 50  0000 L CNN
 F 1 "100n" H 1815 1505 50  0000 L CNN
-F 2 "" H 1738 1400 50  0001 C CNN
+F 2 "Capacitor_SMD:C_1206_3216Metric_Pad1.42x1.75mm_HandSolder" H 1738 1400 50  0001 C CNN
 F 3 "~" H 1700 1550 50  0001 C CNN
 	1    1700 1550
@@
 $EndComp
 $Comp
-L Device:CP C?
+L Device:CP C2
 U 1 1 5E7D4EDD
 P 2100 1550
-F 0 "C?" H 2218 1596 50  0000 L CNN
+F 0 "C2" H 2218 1596 50  0000 L CNN
 F 1 "4.7u" H 2218 1505 50  0000 L CNN
-F 2 "" H 2138 1400 50  0001 C CNN
+F 2 "Capacitor_THT:CP_Radial_D5.0mm_P2.00mm" H 2138 1400 50  0001 C CNN
 F 3 "~" H 2100 1550 50  0001 C CNN
 	1    2100 1550
@@
 Connection ~ 3350 3650
 $Comp
-L Device:C C?
+L Device:C C3
 U 1 1 5E7DCB42
 P 3150 4000
-F 0 "C?" V 2898 4000 50  0000 C CNN
+F 0 "C3" V 2898 4000 50  0000 C CNN
 F 1 "100n" V 2989 4000 50  0000 C CNN
-F 2 "" H 3188 3850 50  0001 C CNN
+F 2 "Capacitor_SMD:C_1206_3216Metric_Pad1.42x1.75mm_HandSolder" H 3188 3850 50  0001 C CNN
 F 3 "~" H 3150 4000 50  0001 C CNN
 	1    3150 4000
@@
 $EndComp
 $Comp
-L power:GND #PWR?
+L power:GND #PWR0105
 U 1 1 5E7DD63C
 P 2950 4150
-F 0 "#PWR?" H 2950 3900 50  0001 C CNN
+F 0 "#PWR0105" H 2950 3900 50  0001 C CNN
 F 1 "GND" H 2955 3977 50  0000 C CNN
 F 2 "" H 2950 4150 50  0001 C CNN
@@
 $EndSheet
 $Comp
-L Connector:Conn_01x02_Male J?
+L Connector:Conn_01x02_Male J5
 U 1 1 5EB20776
 P 3200 3350
-F 0 "J?" V 3050 3300 50  0000 C CNN
+F 0 "J5" V 3050 3300 50  0000 C CNN
 F 1 "Conn_01x02_Male" V 3150 3300 50  0000 C CNN
-F 2 "" H 3200 3350 50  0001 C CNN
+F 2 "Connector_PinHeader_2.54mm:PinHeader_1x02_P2.54mm_Vertical" H 3200 3350 50  0001 C CNN
 F 3 "~" H 3200 3350 50  0001 C CNN
 	1    3200 3350
@@
 	7450 4550 7300 4550
 $Comp
-L Connector:Conn_01x04_Male J?
+L Connector:Conn_01x04_Male J1
 U 1 1 5E7A2BBE
 P 6600 1250
-F 0 "J?" V 6662 1394 50  0000 L CNN
+F 0 "J1" V 6662 1394 50  0000 L CNN
 F 1 "Conn_01x04_Male" V 6753 1394 50  0000 L CNN
-F 2 "" H 6600 1250 50  0001 C CNN
+F 2 "Connector_PinHeader_2.54mm:PinHeader_1x04_P2.54mm_Vertical" H 6600 1250 50  0001 C CNN
 F 3 "~" H 6600 1250 50  0001 C CNN
 	1    6600 1250
@@
 	6600 1450 6600 1700
 $Comp
-L power:GND #PWR?
+L power:GND #PWR0106
 U 1 1 5E7A5BDD
 P 6800 1800
-F 0 "#PWR?" H 6800 1550 50  0001 C CNN
+F 0 "#PWR0106" H 6800 1550 50  0001 C CNN
 F 1 "GND" H 6805 1627 50  0000 C CNN
 F 2 "" H 6800 1800 50  0001 C CNN
@@
 	6800 1600 6800 1800
 $Comp
-L Connector:Conn_01x03_Male J?
+L Connector:Conn_01x03_Male J2
 U 1 1 5E7A8322
 P 8350 1250
-F 0 "J?" V 8412 1394 50  0000 L CNN
+F 0 "J2" V 8412 1394 50  0000 L CNN
 F 1 "Conn_01x03_Male" V 8503 1394 50  0000 L CNN
-F 2 "" H 8350 1250 50  0001 C CNN
+F 2 "Connector_PinHeader_2.54mm:PinHeader_1x03_P2.54mm_Vertical" H 8350 1250 50  0001 C CNN
 F 3 "~" H 8350 1250 50  0001 C CNN
 	1    8350 1250
@@
 USART1_RX
 $Comp
-L power:GND #PWR?
+L power:GND #PWR0107
 U 1 1 5E7A8710
 P 8550 1800
-F 0 "#PWR?" H 8550 1550 50  0001 C CNN
+F 0 "#PWR0107" H 8550 1550 50  0001 C CNN
 F 1 "GND" H 8555 1627 50  0000 C CNN
 F 2 "" H 8550 1800 50  0001 C CNN
@@
 SYS_SWCLK
 $Comp
-L Connector:Conn_01x06_Male J?
+L Connector:Conn_01x06_Male J3
 U 1 1 5E7AD7D5
 P 9950 1250
-F 0 "J?" V 10012 1494 50  0000 L CNN
+F 0 "J3" V 10012 1494 50  0000 L CNN
 F 1 "Conn_01x06_Male" V 10103 1494 50  0000 L CNN
-F 2 "" H 9950 1250 50  0001 C CNN
+F 2 "Connector_PinHeader_2.54mm:PinHeader_1x06_P2.54mm_Vertical" H 9950 1250 50  0001 C CNN
 F 3 "~" H 9950 1250 50  0001 C CNN
 	1    9950 1250
@@
 $EndComp
 $Comp
-L power:GND #PWR?
+L power:GND #PWR0108
 U 1 1 5E7AE29C
 P 10250 1800
-F 0 "#PWR?" H 10250 1550 50  0001 C CNN
+F 0 "#PWR0108" H 10250 1550 50  0001 C CNN
 F 1 "GND" H 10255 1627 50  0000 C CNN
 F 2 "" H 10250 1800 50  0001 C CNN
@@
 Connection ~ 9950 1600
 $Comp
-L Connector:Screw_Terminal_01x03 J?
+L Connector:Screw_Terminal_01x03 J4
 U 1 1 5E7C80AD
 P 4400 1350
-F 0 "J?" V 4364 1162 50  0000 R CNN
+F 0 "J4" V 4364 1162 50  0000 R CNN
 F 1 "Screw_Terminal_01x03" V 4273 1162 50  0000 R CNN
-F 2 "" H 4400 1350 50  0001 C CNN
+F 2 "TerminalBlock:TerminalBlock_bornier-3_P5.08mm" H 4400 1350 50  0001 C CNN
 F 3 "~" H 4400 1350 50  0001 C CNN
 	1    4400 1350
@@
 $EndComp
 $Comp
-L power:+3.3V #PWR?
+L power:+3.3V #PWR0109
 U 1 1 5E7C8DAF
 P 4000 1500
-F 0 "#PWR?" H 4000 1350 50  0001 C CNN
+F 0 "#PWR0109" H 4000 1350 50  0001 C CNN
 F 1 "+3.3V" H 4015 1673 50  0000 C CNN
 F 2 "" H 4000 1500 50  0001 C CNN
@@
 $EndComp
 $Comp
-L power:GND #PWR?
+L power:GND #PWR0110
 U 1 1 5E7C9730
 P 4700 1750
-F 0 "#PWR?" H 4700 1500 50  0001 C CNN
+F 0 "#PWR0110" H 4700 1500 50  0001 C CNN
 F 1 "GND" H 4705 1577 50  0000 C CNN
 F 2 "" H 4700 1750 50  0001 C CNN
@@
 $EndComp
 $Comp
-L power:+5V #PWR?
+L power:+5V #PWR0111
 U 1 1 5E7CA19F
 P 3750 1500
-F 0 "#PWR?" H 3750 1350 50  0001 C CNN
+F 0 "#PWR0111" H 3750 1350 50  0001 C CNN
 F 1 "+5V" H 3765 1673 50  0000 C CNN
 F 2 "" H 3750 1500 50  0001 C CNN

Commit message: Nope, not good
Connections:
- net VU Meter LEDs/-10_dB: now also U1.19 (PA9); no longer U1.22 (PA11)
- net VU Meter LEDs/-20_dB: now also U1.18 (PA8); no longer U1.23 (PA12)
- net VU Meter LEDs/-3_dB: now also U1.23 (PA12); no longer U1.18 (PA8)
- net VU Meter LEDs/-5_dB: now also U1.22 (PA11); no longer U1.19 (PA9)
- net VU Meter LEDs/LEFT: now also U1.8 (PA1); no longer U1.7 (PA0)
- net VU Meter LEDs/RIGHT: now also U1.16 (PB1); no longer U1.8 (PA1)
Changed lines of the file:
@@
 	3800 4950 3600 4950
 Wire Wire Line
-	4900 4850 6550 4850
-Wire Wire Line
-	6550 4750 4900 4750
-Wire Wire Line
-	6550 4650 4900 4650
-Wire Wire Line
-	4900 4550 6550 4550
-Wire Wire Line
-	6550 4450 4900 4450
-Wire Wire Line
 	4900 4350 6550 4350
 Wire Wire Line
@@
 Wire Wire Line
 	4900 3850 6550 3850
-Wire Wire Line
-	4900 3650 5650 3650
-Wire Wire Line
-	5650 3650 5650 3500
-Wire Wire Line
-	5650 3500 7600 3500
-Wire Wire Line
-	7600 3500 7600 4150
-Wire Wire Line
-	7600 4150 7300 4150
-Wire Wire Line
-	4900 3750 5800 3750
-Wire Wire Line
-	5800 3750 5800 3600
-Wire Wire Line
-	5800 3600 7450 3600
-Wire Wire Line
-	7450 3600 7450 4550
-Wire Wire Line
-	7450 4550 7300 4550
 $Comp
 L Connector:Conn_01x04_Male J1
@@
 Wire Wire Line
 	4700 1650 4700 1750
+Wire Wire Line
+	4900 4650 6550 4650
+Wire Wire Line
+	6550 4450 6300 4450
+Wire Wire Line
+	6550 4850 6300 4850
+Wire Wire Line
+	5150 4850 4900 4850
+Wire Wire Line
+	6550 4550 6300 4550
+Wire Wire Line
+	5150 4750 6300 4550
+Wire Wire Line
+	4900 4750 5150 4750
+Wire Wire Line
+	6550 4750 6300 4750
+Wire Wire Line
+	5150 4450 6300 4850
+Wire Wire Line
+	5150 4450 4900 4450
+Wire Wire Line
+	5150 4550 6300 4750
+Wire Wire Line
+	5150 4550 4900 4550
+Wire Wire Line
+	5150 4850 6300 4450
+Wire Wire Line
+	4900 3750 5800 3750
+Wire Wire Line
+	5800 3750 5800 3600
+Wire Wire Line
+	5800 3600 7450 3600
+Wire Wire Line
+	7450 3600 7450 4150
+Wire Wire Line
+	3800 4350 3150 4350
+Wire Wire Line
+	3150 4350 3150 4650
+Wire Wire Line
+	3150 4650 2950 4650
+Wire Wire Line
+	2950 4650 2950 5850
+Wire Wire Line
+	2950 5850 7600 5850
+Wire Wire Line
+	7600 5850 7600 4550
+Wire Wire Line
+	7300 4150 7450 4150
+Wire Wire Line
+	7300 4550 7600 4550
 $EndSCHEMATC

Commit message: Finished PCD Mk.1
Connections:
- net GND: now also C3.1; no longer C3.2
- net I2S_CK: now also J1.2 (Pin_2); no longer J1.4 (Pin_4)
- net I2S_SD: now also J1.4 (Pin_4); no longer J1.2 (Pin_2)
- net at J5.1 (Pin_1), U1.6 (PF2-NRST): now also C3.2; no longer C3.1
- net VU Meter LEDs/+1_dB renamed PN_0
- net VU Meter LEDs/+2_dB renamed NEG_1
- net VU Meter LEDs/+3_dB renamed NEG_2
- net VU Meter LEDs/-10_dB renamed NEG_10
- net VU Meter LEDs/-1_dB renamed POS_2
- net VU Meter LEDs/-20_dB renamed NEG_20
- net VU Meter LEDs/-2_dB renamed POS_3
- net VU Meter LEDs/-3_dB renamed NEG_3
- net VU Meter LEDs/-5_dB renamed NEG_5
- net VU Meter LEDs/-7_dB renamed NEG_7
- net VU Meter LEDs/0_dB renamed POS_1
- net VU Meter LEDs/LEFT renamed L_CH
- net VU Meter LEDs/RIGHT renamed R_CH
Other:
- moved on the sheet: C3, J5, U1
