File: hardware/VU_Meter_LED.sch (KiCad schematic (older format))
At the start: 48 parts

Commit message: First layout
Parts:
- D1, D10, D11, D12, D13, D14, D15, D16, D17, D18, D19, D2, D20, D21, D22, D3, D4, D5, D6, D7, D8, D9: renamed from D?; footprint (none) -> LED_THT:LED_D5.0mm
- Q1, Q10, Q11, Q12, Q13, Q2, Q3, Q4, Q5, Q6, Q7, Q8, Q9: renamed from Q?; footprint Package_TO_SOT_SMD:SOT-23 -> Package_TO_SOT_SMD:SOT-23_Handsoldering
- gave numbers to parts that had none: 13

Commit message: Nope, not good
Parts:
- added R14, R15, R16, R17, R18, R19, R20, R21, R22, R23, R24: 220, Resistor_THT:R_Axial_DIN0207_L6.3mm_D2.5mm_P10.16mm_Horizontal, symbol Device:R
Connections:
- net +5V: now also R14.1, R15.1, R16.1, R17.1, R18.1, R19.1, R20.1, R21.1, R22.1, R23.1, R24.1; no longer Q1.3 (D), Q10.3 (D), Q11.3 (D), Q2.3 (D), Q3.3 (D), Q4.3 (D), Q5.3 (D), Q6.3 (D), Q7.3 (D), Q8.3 (D), Q9.3 (D)
- new net: Q1.3 (D), R14.2
- new net: Q2.3 (D), R15.2
- new net: Q3.3 (D), R16.2
- new net: Q4.3 (D), R17.2
- new net: Q5.3 (D), R18.2
- new net: Q6.3 (D), R19.2
- new net: Q7.3 (D), R20.2
- new net: Q8.3 (D), R21.2
- new net: Q9.3 (D), R22.2
- new net: Q10.3 (D), R23.2
- new net: Q11.3 (D), R24.2
